File: AVR_ISP_SHIELD.kicad_pcb (KiCad board)
At the start: 2 copper layers, 37 parts, among them IC1 ATMEGA328P-P, Y1 Crystal

Commit message: final design
Parts:
- removed W1, W10, W11, W12, W13, W14, W15, W16, W17, W18, W19, W2, W20, W21, W22, W23, W24, W25, W26, W27, W28, W29, W3, W30, W31, W32, W4, W5, W6, W7, W8, W9: TEST_1P, Pin_Headers:Pin_Header_Straight_1x01
- added P1: DIGITAL 2, Pin_Headers:Pin_Header_Straight_1x10, F.Cu at (158.0, 62.7)
- added P2: DIGITAL 1, Pin_Headers:Pin_Header_Straight_1x08, F.Cu at (181.6, 62.7)
- added P3: POWER, Pin_Headers:Pin_Header_Straight_1x08, F.Cu at (145.3, 112.5)
- added P4: ANALOG IN, Pin_Headers:Pin_Header_Straight_1x06, F.Cu at (168.9, 112.5)
- added SW1: SPST, SW_PUSH_6mm:SW_PUSH_SMALL, F.Cu at (126.6, 66.4)
- IC1: footprint ZIF:28tex600 -> 28tex600
- moved Y1 77.1 mm to (155.8, 104.7), turned to 180 degrees
- moved IC1 42.9 mm to (153.0, 86.6)
- moved R1 35.9 mm to (125.1, 112.4)
- moved C2 19.6 mm to (148.2, 104.7), turned to 180 degrees
- moved C1 14.3 mm to (165.9, 104.7), turned to 180 degrees
Routing:
- net 10: track 0.00 -> 108.6 mm
- net GND: track 0.00 -> 94.9 mm
- net VCC: track 0.00 -> 77.6 mm
- net Net-(C1-Pad2): track 0.00 -> 51.7 mm
- net 11: track 0.00 -> 31.8 mm
- net 12: track 0.00 -> 31.2 mm
- net 13: track 0.00 -> 31.1 mm
- net Net-(C2-Pad1): track 0.00 -> 22.7 mm
Other:
- board outline added: 67.5 x 56.4 mm
