File: AVR_ISP_SHIELD.sch (KiCad schematic (older format))
At the start: 41 parts, among them IC1 ATMEGA328P-P, Y1 Crystal

Commit message: final design
Parts:
- removed P?: CONN_01X10, symbol CONN_01X10
- removed P?: CONN_01X06, symbol CONN_01X06
- removed W1, W10, W11, W12, W13, W14, W15, W16, W17, W18, W19, W2, W20, W21, W22, W23, W24, W25, W26, W27, W28, W29, W3, W30, W31, W32, W4, W5, W6, W7, W8, W9: TEST_1P, Pin_Headers:Pin_Header_Straight_1x01, symbol TEST_1P
- added P1: DIGITAL 2, Pin_Headers:Pin_Header_Straight_1x10, symbol CONN_01X08_D2_UNO-RESCUE-AVR_ISP_SHIELD
- added P4: ANALOG IN, Pin_Headers:Pin_Header_Straight_1x06, symbol CONN_01X06_ANALOG_IN_UNO
- added SW1: SPST, SW_PUSH_6mm:SW_PUSH_SMALL, symbol SPST
- P2: renamed from P?; value CONN_01X08_D1_UNO -> DIGITAL 1; footprint (none) -> Pin_Headers:Pin_Header_Straight_1x08
- P3: renamed from P?; value CONN_01X08_POWER_UNO -> POWER; footprint (none) -> Pin_Headers:Pin_Header_Straight_1x08; symbol CONN_01X08_POWER_UNO -> CONN_01X08_POWER_UNO-RESCUE-AVR_ISP_SHIELD
Connections:
- net 10: now also P1.3 (10), SW1.2
- net 11: now also P1.4 (11)
- net 12: now also P1.5 (12)
- net 13: now also P1.6 (13)
- net GND: now also P3.2 (GND), P3.3 (GND), P1.7 (GND), SW1.1
- net VCC: now also P3.4 (5v)
- no-connect marks 0 -> 24
Other:
- moved on the sheet: P3
